Commit message: scout_description first working version

File: scout/scout_description/urdf/scout_mini.xacro (robot description, xacro)
@@ -2,70 +2,38 @@
 <robot name="scout_mini"
     xmlns:xacro="http://ros.org/wiki/xacro">
-    <xacro:arg name="robot_namespace" default="/" />
     <xacro:arg name="urdf_extras" default="empty.urdf" />
-    <xacro:include filename="$(find scout_description)/urdf/scout_mini_wheel_1.xacro" />
-    <xacro:include filename="$(find scout_description)/urdf/scout_mini_wheel_2.xacro" />
-    <xacro:include filename="$(find scout_description)/urdf/scout_mini_wheel_3.xacro" />
-    <xacro:include filename="$(find scout_description)/urdf/scout_mini_wheel_4.xacro" />
-    <!-- Variables -->
-    <xacro:property name="M_PI" value="3.14159"/>
     <!-- Vehicle Geometries -->
-    <xacro:property name="base_x_size" value="0.6200000" />
-    <xacro:property name="base_y_size" value="0.585000" />
-    <xacro:property name="base_z_size" value="0.235000" />
     <xacro:property name="wheelbase" value="0.3132556"/>
-   <xacro:property name="track" value="0.4563536" />
-   <xacro:property name="wheel_vertical_offset" value="-0.077" />
-<!--    <xacro:property name="track" value="0.3426" />
-    <xacro:property name="wheelbase" value="0.3181"/>
-    <xacro:property name="wheel_vertical_offset" value="-0.160000047342231" />-->
-    <xacro:property name="wheel_length" value="0.8e-01" />
-    <xacro:property name="wheel_radius" value="1.600e-01" />
+    <xacro:property name="track" value="0.4563536" />
+    <xacro:property name="wheel_vertical_offset" value="-0.077" />
+    <!-- For testing, hang the robot up in the air
+    <link name="world" />
+    <joint name="world_to_base_link" type="fixed">
+        <origin xyz="0 0 0.5" rpy="0 0 0" />
+        <parent link="world"/>
+        <child link="base_link"/>
+    </joint> -->
     <!-- Base link -->
     <link name="base_link">
         <visual>
-            <!--origin xyz="-0.0145261552504705 0.0231316650320557 0.00586280190939592" rpy="0 0 0" /-->
-            <origin xyz="0.015 0.0231316650320557 0" rpy="0 0 0"/>
-            <!--<origin
-              xyz="-0.0145261552504705 0.0231316650320557 0.00586280190939592"
-              rpy="0 0 0" />-->
+            <origin xyz="0.015 0.0231316650320557 0" rpy="1.57 0 0"/>
             <geometry>
-                <mesh filename="package://scout_description/meshes/scout_mini_base_link.STL" />
+                <mesh filename="package://scout_description/meshes/scout_mini_base_link.dae" />
             </geometry>
         </visual>
         <collision>
-          <!--origin
-            xyz="-0.0145261552504705 0.0231316650320557 0.00586280190939592"
-            rpy="0 0 0" /-->
-            <origin xyz="0.015 0.0231316650320557 0" rpy="0 0 0"/>
+            <origin xyz="0.015 0.0231316650320557 0" rpy="1.57 0 0"/>
           <geometry>
             <mesh
-              filename="package://scout_description/meshes/scout_mini_base_link.STL" />
+              filename="package://scout_description/meshes/scout_mini_base_link.dae" />
           </geometry>
         </collision>
     </link>
-    <!-- <joint name="chassis_link_joint" type="fixed">
-        <origin xyz="0 0 ${wheel_radius - wheel_vertical_offset}" rpy="0 0 0" />
-        <parent link="base_link" />
-        <child link="chassis_link" />
-    </joint> -->
     <link name="inertial_link">
         <inertial>
-            <!--mass value="44.3898489950015" /-->
             <mass value="132.3898489950015" />
-            <!-- <mass value="50" /> -->
-            <!-- <origin xyz="-0.00065 -0.085 0.062" />
-            <inertia ixx="0.6022" ixy="-0.02364" ixz="-0.1197" iyy="1.7386" iyz="-0.001544" izz="2.0296" /> -->
             <origin xyz="0.015 0.0231316650320557 0" />
-            <!--<origin
-              xyz="-0.0145261552504705 0.0231316650320557 0.00586280190939592"
-              rpy="0 0 0" />-->
-            <inertia ixx="0.185196122711036"
-            ixy="4.30144213829512E-08"
-            ixz="5.81037523686401E-08"
-            iyy="0.364893736238929"
-            iyz="-0.000386720198091934"
-            izz="0.223868521722778" />
-            <!--<inertia ixx="2.288641" ixy="0" ixz="0" iyy="5.103976" iyz="0" izz="3.431465" />-->
+            <inertia ixx="0.185196122711036" ixy="4.30144213829512E-08" ixz="5.81037523686401E-08"
+            iyy="0.364893736238929" iyz="-0.000386720198091934" izz="0.223868521722778" />
         </inertial>
     </link>
@@ -75,29 +43,106 @@
         <child link="inertial_link" />
     </joint>
-    <!-- For testing, hang the robot up in the air -->
-    <!-- <link name="world" />
-    <joint name="world_to_base_link=" type="fixed">
-        <origin xyz="0 0 0.5" rpy="0 0 0" />
-        <parent link="world"/>
-        <child link="base_link"/>
-    </joint> -->
     <!-- Scout wheel macros -->
-    <!-- wheel labeled from 0 to 3, conter-clockwise, starting from front right wheel -->
-    <!-- motor 1 and 2 (left side) are mechanically installed in a reversed direction -->
-    <xacro:scout_mini_wheel_1 wheel_prefix="rear_right">
+    <link name="front_right_wheel_link">
+        <inertial>
+            <mass value="3" />
+            <origin xyz="0 0 0" />
+            <inertia ixx="0.7171" ixy="0" ixz="0" iyy="0.7171" iyz="0" izz="0.1361" />
+        </inertial>
+        <visual>
+            <origin xyz="0 0 0" rpy="0 0 0" />
+            <geometry>
+                <mesh filename="package://scout_description/meshes/wheel.dae" />
+            </geometry>
+        </visual>
+        <collision>
+          <origin xyz="0 0 0" rpy="0 0 0" />
+          <geometry>
+            <mesh filename="package://scout_description/meshes/wheel.dae" />
+          </geometry>
+        </collision>
+    </link>
+    <joint name="front_right_wheel" type="continuous">
+        <origin xyz="${wheelbase/2} ${track/2} ${wheel_vertical_offset}" rpy="0 1.57 0" />
+        <parent link="base_link"/>
+        <child link="front_right_wheel_link"/>
+        <axis xyz="0 0 -1" rpy="0 0 0" />
+    </joint>
+    <link name="front_left_wheel_link">
+        <inertial>
+            <mass value="3" />
+            <origin xyz="0 0 0" />
+            <inertia ixx="0.7171" ixy="0" ixz="0" iyy="0.7171" iyz="0" izz="0.1361" />
+        </inertial>
+        <visual>
+            <origin xyz="0 0 0" rpy="0 0 0" />
+            <geometry>
+                <mesh filename="package://scout_description/meshes/wheel.dae" />
+            </geometry>
+        </visual>
+        <collision>
+          <origin xyz="0 0 0" rpy="0 0 0" />
+          <geometry>
+            <mesh filename="package://scout_description/meshes/wheel.dae" />
+          </geometry>
+        </collision>
+    </link>
+    <joint name="front_left_wheel" type="continuous">
+        <origin xyz="${-wheelbase/2} ${track/2} ${wheel_vertical_offset}" rpy="0 -1.57 0" />
+        <parent link="base_link"/>
+        <child link="front_left_wheel_link"/>
+        <axis xyz="0 0 1" rpy="0 0 0" />
+    </joint>
+    <link name="rear_right_wheel_link">
+        <inertial>
+            <mass value="3" />
+            <origin xyz="0 0 0" />
+            <inertia ixx="0.7171" ixy="0" ixz="0" iyy="0.7171" iyz="0" izz="0.1361" />
+        </inertial>
+        <visual>
+            <origin xyz="0 0 0" rpy="0 0 0" />
+            <geometry>
+                <mesh filename="package://scout_description/meshes/wheel.dae" />
+            </geometry>
+        </visual>
+        <collision>
+          <origin xyz="0 0 0" rpy="0 0 0" />
+          <geometry>
+            <mesh filename="package://scout_description/meshes/wheel.dae" />
+          </geometry>
+        </collision>
+    </link>
+    <joint name="rear_right_wheel" type="continuous">
         <origin xyz="${wheelbase/2} ${-track/2} ${wheel_vertical_offset}" rpy="0 1.57 0" />
-    </xacro:scout_mini_wheel_1>
-    <xacro:scout_mini_wheel_2 wheel_prefix="front_right">
-        <origin xyz="${wheelbase/2} ${track/2} ${wheel_vertical_offset}" rpy="0 1.57 0" />
-    </xacro:scout_mini_wheel_2>
-    <xacro:scout_mini_wheel_3 wheel_prefix="front_left">
-        <origin xyz="${-wheelbase/2} ${track/2} ${wheel_vertical_offset}" rpy="0 -1.57 0" />
-    </xacro:scout_mini_wheel_3>
-    <xacro:scout_mini_wheel_4 wheel_prefix="rear_left">
+        <parent link="base_link"/>
+        <child link="rear_right_wheel_link"/>
+        <axis xyz="0 0 -1" rpy="0 0 0" />
+    </joint>
+    <link name="rear_left_wheel_link">
+        <inertial>
+            <mass value="3" />
+            <origin xyz="0 0 0" />
+            <inertia ixx="0.7171" ixy="0" ixz="0" iyy="0.7171" iyz="0" izz="0.1361" />
+        </inertial>
+        <visual>
+            <origin xyz="0 0 0" rpy="0 0 0" />
+            <geometry>
+                <mesh filename="package://scout_description/meshes/wheel.dae" />
+            </geometry>
+        </visual>
+        <collision>
+          <origin xyz="0 0 0" rpy="0 0 0" />
+          <geometry>
+            <mesh filename="package://scout_description/meshes/wheel.dae" />
+          </geometry>
+        </collision>
+    </link>
+    <joint name="rear_left_wheel" type="continuous">
         <origin xyz="${-wheelbase/2} ${-track/2} ${wheel_vertical_offset}" rpy="0 -1.57 0" />
-    </xacro:scout_mini_wheel_4>
+        <parent link="base_link"/>
+        <child link="rear_left_wheel_link"/>
+        <axis xyz="0 0 1" rpy="0 0 0" />
+    </joint>
     <!-- Additional definitions -->
     <xacro:include filename="$(arg urdf_extras)" />
-    <!-- Gazebo definitions  -->
-    <xacro:include filename="$(find scout_description)/urdf/scout_mini.gazebo" />
 </robot>

File: scout/scout_description/urdf/scout_v2.xacro (robot description, xacro)
@@ -2,8 +2,5 @@
 <robot name="scout_v2"
     xmlns:xacro="http://ros.org/wiki/xacro">
-    <xacro:arg name="robot_namespace" default="/" />
     <xacro:arg name="urdf_extras" default="empty.urdf" />
-    <xacro:include filename="$(find scout_description)/urdf/scout_wheel_type1.xacro" />
-    <xacro:include filename="$(find scout_description)/urdf/scout_wheel_type2.xacro" />
     <!-- Variables -->
     <xacro:property name="M_PI" value="3.14159"/>
@@ -17,4 +14,11 @@
     <xacro:property name="wheel_length" value="1.1653e-01" />
     <xacro:property name="wheel_radius" value="1.6459e-01" />
+    <!-- For testing, hang the robot up in the air
+    <link name="world" />
+    <joint name="world_to_base_link" type="fixed">
+        <origin xyz="0 0 0.5" rpy="0 0 0" />
+        <parent link="world"/>
+        <child link="base_link"/>
+    </joint> -->
     <!-- Base link -->
     <link name="base_link">
@@ -38,15 +42,7 @@
         </collision>
     </link>
-    <!-- <joint name="chassis_link_joint" type="fixed">
-        <origin xyz="0 0 ${wheel_radius - wheel_vertical_offset}" rpy="0 0 0" />
-        <parent link="base_link" />
-        <child link="chassis_link" />
-    </joint> -->
     <link name="inertial_link">
         <inertial>
             <mass value="50" />
-            <!-- <mass value="50" /> -->
-            <!-- <origin xyz="-0.00065 -0.085 0.062" />
-            <inertia ixx="0.6022" ixy="-0.02364" ixz="-0.1197" iyy="1.7386" iyz="-0.001544" izz="2.0296" /> -->
             <origin xyz="0.0 0.0 0.0" />
             <inertia ixx="2.288641" ixy="0" ixz="0" iyy="5.103976" iyz="0" izz="3.431465" />
@@ -58,29 +54,126 @@
         <child link="inertial_link" />
     </joint>
-    <!-- For testing, hang the robot up in the air -->
-    <!-- <link name="world" />
-    <joint name="world_to_base_link=" type="fixed">
-        <origin xyz="0 0 0.5" rpy="0 0 0" />
-        <parent link="world"/>
-        <child link="base_link"/>
-    </joint> -->
     <!-- Scout wheel macros -->
-    <!-- wheel labeled from 0 to 3, conter-clockwise, starting from front right wheel -->
-    <!-- motor 1 and 2 (left side) are mechanically installed in a reversed direction -->
-    <xacro:scout_wheel_type1 wheel_prefix="front_right">
+    <link name="front_right_wheel_link">
+        <inertial>
+            <mass value="8" />
+            <origin xyz="0 0 0" />
+            <inertia ixx="0.1171" ixy="0" ixz="0" iyy="0.1361" iyz="0" izz="0.1171" />
+        </inertial>
+        <visual>
+            <origin xyz="0 0 0" rpy="0 0 0" />
+            <geometry>
+                <mesh filename="package://scout_description/meshes/wheel_type1.dae" />
+            </geometry>
+        </visual>
+        <collision>
+            <origin xyz="0 0 0" rpy="${M_PI/2} 0 0" />
+            <geometry>
+                <cylinder length="${wheel_length}" radius="${wheel_radius}" />
+            </geometry>
+            <contact>
+                <ode>
+                    <min_depth>0.001</min_depth>
+                </ode>
+            </contact>
+        </collision>
+    </link>
+    <joint name="front_right_wheel" type="continuous">
         <origin xyz="${wheelbase/2} ${-track/2} ${wheel_vertical_offset}" rpy="3.14 0 0" />
-    </xacro:scout_wheel_type1>
-    <xacro:scout_wheel_type2 wheel_prefix="front_left">
+        <parent link="base_link"/>
+        <child link="front_right_wheel_link"/>
+        <axis xyz="0 -1 0" rpy="0 0 0" />
+    </joint>
+    <link name="rear_left_wheel_link">
+        <inertial>
+            <mass value="8" />
+            <origin xyz="0 0 0" />
+            <inertia ixx="0.1171" ixy="0" ixz="0" iyy="0.1361" iyz="0" izz="0.1171" />
+        </inertial>
+        <visual>
+            <origin xyz="0 0 0" rpy="0 0 0" />
+            <geometry>
+                <mesh filename="package://scout_description/meshes/wheel_type1.dae" />
+            </geometry>
+        </visual>
+        <collision>
+            <origin xyz="0 0 0" rpy="${M_PI/2} 0 0" />
+            <geometry>
+                <cylinder length="${wheel_length}" radius="${wheel_radius}" />
+            </geometry>
+            <contact>
+                <ode>
+                    <min_depth>0.001</min_depth>
+                </ode>
+            </contact>
+        </collision>
+    </link>
+    <joint name="rear_left_wheel" type="continuous">
+        <origin xyz="${-wheelbase/2} ${track/2} ${wheel_vertical_offset}" rpy="0 0 0" />
+        <parent link="base_link"/>
+        <child link="rear_left_wheel_link"/>
+        <axis xyz="0 1 0" rpy="0 0 0" />
+    </joint>
+    <link name="front_left_wheel_link">
+        <inertial>
+            <mass value="8" />
+            <origin xyz="0 0 0" />
+            <inertia ixx="0.1171" ixy="0" ixz="0" iyy="0.1361" iyz="0" izz="0.1171" />
+        </inertial>
+        <visual>
+            <origin xyz="0 0 0" rpy="0 0 0" />
+            <geometry>
+                <mesh filename="package://scout_description/meshes/wheel_type1.dae" />
+            </geometry>
+        </visual>
+        <collision>
+            <origin xyz="0 0 0" rpy="${M_PI/2} 0 0" />
+            <geometry>
+                <cylinder length="${wheel_length}" radius="${wheel_radius}" />
+            </geometry>
+            <contact>
+                <ode>
+                    <min_depth>0.001</min_depth>
+                </ode>
+            </contact>
+        </collision>
+    </link>
+    <joint name="front_left_wheel" type="continuous">
         <origin xyz="${wheelbase/2} ${track/2} ${wheel_vertical_offset}" rpy="0 0 0" />
-    </xacro:scout_wheel_type2>
-    <xacro:scout_wheel_type1 wheel_prefix="rear_left">
-        <origin xyz="${-wheelbase/2} ${track/2} ${wheel_vertical_offset}" rpy="0 0 0" />
-    </xacro:scout_wheel_type1>
-    <xacro:scout_wheel_type2 wheel_prefix="rear_right">
+        <parent link="base_link"/>
+        <child link="front_left_wheel_link"/>
+        <axis xyz="0 1 0" rpy="0 0 0" />
+    </joint>
+    <link name="rear_right_wheel_link">
+        <inertial>
+            <mass value="8" />
+            <origin xyz="0 0 0" />
+            <inertia ixx="0.1171" ixy="0" ixz="0" iyy="0.1361" iyz="0" izz="0.1171" />
+        </inertial>
+        <visual>
+            <origin xyz="0 0 0" rpy="0 0 0" />
+            <geometry>
+                <mesh filename="package://scout_description/meshes/wheel_type1.dae" />
+            </geometry>
+        </visual>
+        <collision>
+            <origin xyz="0 0 0" rpy="${M_PI/2} 0 0" />
+            <geometry>
+                <cylinder length="${wheel_length}" radius="${wheel_radius}" />
+            </geometry>
+            <contact>
+                <ode>
+                     <min_depth>0.001</min_depth>
+                </ode>
+            </contact>
+        </collision>
+    </link>
+    <joint name="rear_right_wheel" type="continuous">
         <origin xyz="${-wheelbase/2} ${-track/2} ${wheel_vertical_offset}" rpy="3.14 0 0" />
-    </xacro:scout_wheel_type2>
+        <parent link="base_link"/>
+        <child link="rear_right_wheel_link"/>
+        <axis xyz="0 -1 0" rpy="0 0 0" />
+    </joint>
     <!-- Additional definitions -->
     <xacro:include filename="$(arg urdf_extras)" />
-    <!-- Gazebo definitions  -->
-    <xacro:include filename="$(find scout_description)/urdf/scout_v2.gazebo" />
 </robot>

Commit message: new models including sensors

File: scout/scout_description/urdf/scout_mini.xacro (robot description, xacro)
@@ -2,5 +2,5 @@
 <robot name="scout_mini"
     xmlns:xacro="http://ros.org/wiki/xacro">
-    <xacro:arg name="urdf_extras" default="empty.urdf" />
+    <xacro:arg name="urdf_extras" default="scout_mini_extras.urdf" />
     <!-- Vehicle Geometries -->
     <xacro:property name="wheelbase" value="0.3132556"/>
@@ -17,5 +17,5 @@
     <link name="base_link">
         <visual>
-            <origin xyz="0.015 0.0231316650320557 0" rpy="1.57 0 0"/>
+            <origin xyz="0.015 0.0231316650320557 0" rpy="1.57 0 -1.57"/>
             <geometry>
                 <mesh filename="package://scout_description/meshes/scout_mini_base_link.dae" />
@@ -23,5 +23,5 @@
         </visual>
         <collision>
-            <origin xyz="0.015 0.0231316650320557 0" rpy="1.57 0 0"/>
+            <origin xyz="0.015 0.0231316650320557 0" rpy="1.57 0 -1.57"/>
           <geometry>
             <mesh
@@ -64,5 +64,5 @@
     </link>
     <joint name="front_right_wheel" type="continuous">
-        <origin xyz="${wheelbase/2} ${track/2} ${wheel_vertical_offset}" rpy="0 1.57 0" />
+        <origin xyz="${track/2} ${-wheelbase/2} ${wheel_vertical_offset}" rpy="1.57 0 0" />
         <parent link="base_link"/>
         <child link="front_right_wheel_link"/>
@@ -89,5 +89,5 @@
     </link>
     <joint name="front_left_wheel" type="continuous">
-        <origin xyz="${-wheelbase/2} ${track/2} ${wheel_vertical_offset}" rpy="0 -1.57 0" />
+        <origin xyz="${track/2} ${wheelbase/2} ${wheel_vertical_offset}" rpy="-1.57 0 0" />
         <parent link="base_link"/>
         <child link="front_left_wheel_link"/>
@@ -114,5 +114,5 @@
     </link>
     <joint name="rear_right_wheel" type="continuous">
-        <origin xyz="${wheelbase/2} ${-track/2} ${wheel_vertical_offset}" rpy="0 1.57 0" />
+        <origin xyz="${-track/2} ${-wheelbase/2} ${wheel_vertical_offset}" rpy="1.57 0 0" />
         <parent link="base_link"/>
         <child link="rear_right_wheel_link"/>
@@ -139,5 +139,5 @@
     </link>
     <joint name="rear_left_wheel" type="continuous">
-        <origin xyz="${-wheelbase/2} ${-track/2} ${wheel_vertical_offset}" rpy="0 -1.57 0" />
+        <origin xyz="${-track/2} ${wheelbase/2} ${wheel_vertical_offset}" rpy="-1.57 0 0" />
         <parent link="base_link"/>
         <child link="rear_left_wheel_link"/>

File: scout/scout_description/urdf/scout_v2.xacro (robot description, xacro)
@@ -2,5 +2,5 @@
 <robot name="scout_v2"
     xmlns:xacro="http://ros.org/wiki/xacro">
-    <xacro:arg name="urdf_extras" default="empty.urdf" />
+    <xacro:arg name="urdf_extras" default="scout_v2_extras.urdf" />
     <!-- Variables -->
     <xacro:property name="M_PI" value="3.14159"/>

Commit message: Add the twist_mux for implementing the dead-man switch, add SLAM functionality, clear the xacro files and create a new rviz file for a simpler and clear view on rviz

File: scout/scout_description/urdf/scout_mini.xacro (robot description, xacro)
@@ -1,5 +1,4 @@
 <?xml version="1.0"?>
-<robot name="scout_mini"
-    xmlns:xacro="http://ros.org/wiki/xacro">
+<robot name="scout_mini" xmlns:xacro="http://ros.org/wiki/xacro">
     <xacro:arg name="urdf_extras" default="scout_mini_extras.urdf" />
     <!-- Vehicle Geometries -->
@@ -7,11 +6,4 @@
     <xacro:property name="track" value="0.4563536" />
     <xacro:property name="wheel_vertical_offset" value="-0.077" />
-    <!-- For testing, hang the robot up in the air
-    <link name="world" />
-    <joint name="world_to_base_link" type="fixed">
-        <origin xyz="0 0 0.5" rpy="0 0 0" />
-        <parent link="world"/>
-        <child link="base_link"/>
-    </joint> -->
     <!-- Base link -->
     <link name="base_link">
@@ -144,4 +136,47 @@
         <axis xyz="0 0 1" rpy="0 0 0" />
     </joint>
+    <!-- plug-in -->
+    <plugin name='scout_mini_joint_state' filename='libgazebo_ros_joint_state_publisher.so'>
+      <ros>
+        <namespace>/robot_namespace</namespace>
+        <remapping>~/out:=joint_states</remapping>
+      </ros>
+      <update_rate>50</update_rate>
+      <joint_name>front_right_wheel</joint_name>
+      <joint_name>front_left_wheel</joint_name>
+      <joint_name>rear_right_wheel</joint_name>
+      <joint_name>rear_left_wheel</joint_name>
+    </plugin>
+    <plugin name='skid_steer_drive' filename='libgazebo_ros_diff_drive.so'>
+      <!-- topics & remappings -->
+      <ros>
+        <namespace>/robot_namespace</namespace>
+      </ros>
+      <!-- Update rate -->
+      <update_rate>50</update_rate>
+      <!-- Number of wheel pairs -->
+      <num_wheel_pairs>2</num_wheel_pairs>
+      <!-- front wheels -->
+      <left_joint>front_left_wheel</left_joint>
+      <right_joint>front_right_wheel</right_joint>
+      <!-- rear wheels-->
+      <left_joint>rear_left_wheel</left_joint>
+      <right_joint>rear_right_wheel</right_joint>
+      <!-- kinematics -->
+      <wheel_separation>0.490</wheel_separation>
+      <wheel_separation>0.490</wheel_separation>
+      <wheel_diameter>0.160</wheel_diameter>
+      <wheel_diameter>0.160</wheel_diameter>
+      <!-- limits -->
+      <max_wheel_torque>20</max_wheel_torque>
+      <max_wheel_acceleration>1.0</max_wheel_acceleration>
+      <!-- output -->
+      <publish_odom>true</publish_odom>
+      <publish_odom_tf>true</publish_odom_tf>
+      <publish_wheel_tf>true</publish_wheel_tf>
+      <odometry_frame>odom</odometry_frame>
+      <odometry_topic>odom</odometry_topic>
+      <robot_base_frame>base_link</robot_base_frame>
+    </plugin>
     <!-- Additional definitions -->
     <xacro:include filename="$(arg urdf_extras)" />

File: scout/scout_description/urdf/scout_mini_extras.urdf (robot description, URDF)
Before this commit: robot None, 3 links, 3 joints
Joints:
- joint scan_joint: axis (none) -> 0 1 0
