Commit message: Fixed scout_mini wheel position

File: scout/scout_description/urdf/scout_mini.xacro (robot description, xacro)
@@ -2,13 +2,8 @@
 <robot name="scout_mini" xmlns:xacro="http://ros.org/wiki/xacro">
     <!-- Vehicle Geometries -->
-    <xacro:property name="wheelbase"
-        value="0.3132556" />
-    <xacro:property name="track" value="0.4563536" />
-    <xacro:property
-        name="wheel_vertical_offset" value="-0.077" />
     <!-- Base link -->
     <link name="base_link">
         <visual>
-            <origin xyz="0.015 0.0231316650320557 0" rpy="1.57 0 -1.57" />
+            <origin xyz="0 0 0" rpy="1.57 0 -1.57" />
             <geometry>
                 <mesh
@@ -17,5 +12,5 @@
         </visual>
         <collision>
-            <origin xyz="0.015 0.0231316650320557 0" rpy="1.57 0 -1.57" />
+            <origin xyz="0 0 0" rpy="1.57 0 -1.57" />
             <geometry>
                 <mesh
@@ -28,5 +23,5 @@
         <inertial>
             <mass value="132.3898489950015" />
-            <origin xyz="0.015 0.0231316650320557 0" />
+            <origin xyz=" 0 0 0" />
             <inertia ixx="0.185196122711036" ixy="4.30144213829512E-08" ixz="5.81037523686401E-08"
                 iyy="0.364893736238929" iyz="-0.000386720198091934" izz="0.223868521722778" />
@@ -62,5 +57,5 @@
     <joint
         name="front_right_wheel" type="continuous">
-        <origin xyz="${track/2} ${-wheelbase/2} ${wheel_vertical_offset}" rpy="1.57 0 0" />
+        <origin rpy="1.57 0 0" xyz="0.2319755 -0.2082515 -0.099998" />
         <parent link="base_link" />
         <child link="front_right_wheel_link" />
@@ -88,5 +83,5 @@
     <joint
         name="front_left_wheel" type="continuous">
-        <origin xyz="${track/2} ${wheelbase/2} ${wheel_vertical_offset}" rpy="-1.57 0 0" />
+        <origin rpy="-1.57 0 0" xyz="0.2319755 0.2082515 -0.100998" />
         <parent link="base_link" />
         <child link="front_left_wheel_link" />
@@ -114,5 +109,5 @@
     <joint
         name="rear_right_wheel" type="continuous">
-        <origin xyz="${-track/2} ${-wheelbase/2} ${wheel_vertical_offset}" rpy="1.57 0 0" />
+        <origin rpy="1.57 0 0" xyz="-0.2319755 -0.2082515 -0.099998" />
         <parent link="base_link" />
         <child link="rear_right_wheel_link" />
@@ -140,5 +135,5 @@
     <joint
         name="rear_left_wheel" type="continuous">
-        <origin xyz="${-track/2} ${wheelbase/2} ${wheel_vertical_offset}" rpy="-1.57 0 0" />
+        <origin rpy="-1.57 0 0" xyz="-0.2319755 0.2082515 -0.100998" />
         <parent link="base_link" />
         <child link="rear_left_wheel_link" />
