Commit message: Revert "Add bunker and scout_mini for jazzy and gazebo harmonic"
This reverts commit 35988f9ddacb2aa28f5d58a0834fa076c9a7dad3.

File: bunker/bunker_description/urdf/bunker.xacro (robot description, xacro)
@@ -1,5 +1,4 @@
 <?xml version="1.0"?>
-<robot name="bunker"
-    xmlns:xacro="http://www.ros.org/wiki/xacro">
+<robot name="bunker" xmlns:xacro="http://www.ros.org/wiki/xacro">
     <!-- Vehicle Geometries -->
     <!-- Base link -->
@@ -8,5 +7,6 @@
             <origin xyz="0.53 -0.392 -0.358" rpy="1.57 0 3.14" />
             <geometry>
-                <mesh filename="package://bunker_description/meshes/bunker.stl" scale="0.001 0.001 0.001" />
+                <mesh filename="package://bunker_description/meshes/bunker.stl"
+                    scale="0.001 0.001 0.001" />
             </geometry>
             <material name="">
@@ -17,5 +17,6 @@
             <origin xyz="0.53 -0.392 -0.358" rpy="1.57 0 3.14" />
             <geometry>
-                <mesh filename="package://bunker_description/meshes/bunker.stl" scale="0.001 0.001 0.001" />
+                <mesh filename="package://bunker_description/meshes/bunker.stl"
+                    scale="0.001 0.001 0.001" />
             </geometry>
         </collision>
@@ -25,5 +26,6 @@
             <origin xyz="0.0212410555532523 0.00475458359568469 -0.127580557949736" rpy="0 0 0" />
             <mass value="22" />
-            <inertia ixx="0.607716166684979" ixy="1.92178193996147E-05" ixz="-0.036532069356182" iyy="1.70041426855404" iyz="2.16963122007266E-05" izz="1.84232351935185" />
+            <inertia ixx="0.607716166684979" ixy="1.92178193996147E-05" ixz="-0.036532069356182"
+                iyy="1.70041426855404" iyz="2.16963122007266E-05" izz="1.84232351935185" />
         </inertial>
     </link>
@@ -36,5 +38,7 @@
             <origin xyz="0 -1.38777878078145E-17 -0.0719999999999999" rpy="0 0 0" />
             <mass value="0.392034219968119" />
-            <inertia ixx="0.000378440530116381" ixy="5.60822736805661E-21" ixz="3.04207802822425E-20" iyy="0.000378440530116381" iyz="-7.56626980356474E-21" izz="0.000710150518820894" />
+            <inertia ixx="0.000378440530116381" ixy="5.60822736805661E-21"
+                ixz="3.04207802822425E-20"
+                iyy="0.000378440530116381" iyz="-7.56626980356474E-21" izz="0.000710150518820894" />
         </inertial>
         <visual>
@@ -62,5 +66,7 @@
             <origin xyz="-1.74279013442913E-08 5.87093572021469E-08 -0.0720000000000001" rpy="0 0 0" />
             <mass value="0.190328287901002" />
-            <inertia ixx="6.58750963981394E-05" ixy="-1.46558944641469E-09" ixz="-8.34967331718859E-12" iyy="6.58795984671517E-05" iyz="-2.4786046130206E-12" izz="0.000112721820875598" />
+            <inertia ixx="6.58750963981394E-05" ixy="-1.46558944641469E-09"
+                ixz="-8.34967331718859E-12"
+                iyy="6.58795984671517E-05" iyz="-2.4786046130206E-12" izz="0.000112721820875598" />
         </inertial>
         <visual>
@@ -88,5 +94,6 @@
             <origin xyz="1.66533453693773E-16 4.16333634234434E-17 -0.0720000000000002" rpy="0 0 0" />
             <mass value="0.271192811687251" />
-            <inertia ixx="0.000179574259018481" ixy="1.15789498120549E-20" ixz="1.3563351843978E-21" iyy="0.000179574259018481" iyz="6.0369822309622E-23" izz="0.000332594534732139" />
+            <inertia ixx="0.000179574259018481" ixy="1.15789498120549E-20" ixz="1.3563351843978E-21"
+                iyy="0.000179574259018481" iyz="6.0369822309622E-23" izz="0.000332594534732139" />
         </inertial>
         <visual>
@@ -114,5 +121,7 @@
             <origin xyz="3.44025652177504E-05 -2.66346274915008E-05 -0.0701504149473696" rpy="0 0 0" />
             <mass value="0.245835028330933" />
-            <inertia ixx="0.000105254202004996" ixy="1.32328029886322E-08" ixz="3.84294589102693E-11" iyy="0.000105248656147198" iyz="-1.41155611914915E-11" izz="0.000173280771745758" />
+            <inertia ixx="0.000105254202004996" ixy="1.32328029886322E-08"
+                ixz="3.84294589102693E-11"
+                iyy="0.000105248656147198" iyz="-1.41155611914915E-11" izz="0.000173280771745758" />
         </inertial>
         <visual>
@@ -140,5 +149,7 @@
             <origin xyz="-1.66533453693773E-16 0 0.072" rpy="0 0 0" />
             <mass value="0.392034219968119" />
-            <inertia ixx="0.000378440530116381" ixy="3.37302217863781E-21" ixz="2.71827270955143E-20" iyy="0.000378440530116381" iyz="-7.32821644893157E-21" izz="0.000710150518820894" />
+            <inertia ixx="0.000378440530116381" ixy="3.37302217863781E-21"
+                ixz="2.71827270955143E-20"
+                iyy="0.000378440530116381" iyz="-7.32821644893157E-21" izz="0.000710150518820894" />
         </inertial>
         <visual>
@@ -166,5 +177,7 @@
             <origin xyz="-1.74279017328693E-08 5.87093572160247E-08 0.0720000000000002" rpy="0 0 0" />
             <mass value="0.190328287901002" />
-            <inertia ixx="6.58750963981394E-05" ixy="-1.46558944642761E-09" ixz="-8.34967332343028E-12" iyy="6.58795984671517E-05" iyz="-2.47860459929511E-12" izz="0.000112721820875598" />
+            <inertia ixx="6.58750963981394E-05" ixy="-1.46558944642761E-09"
+                ixz="-8.34967332343028E-12"
+                iyy="6.58795984671517E-05" iyz="-2.47860459929511E-12" izz="0.000112721820875598" />
         </inertial>
         <visual>
@@ -192,5 +205,6 @@
             <origin xyz="-1.38777878078145E-16 -4.85722573273506E-17 0.0720000000000003" rpy="0 0 0" />
             <mass value="0.27119281168725" />
-            <inertia ixx="0.00017957425901848" ixy="6.28960386226657E-21" ixz="2.14010788664762E-21" iyy="0.00017957425901848" iyz="1.27709655724716E-22" izz="0.000332594534732139" />
+            <inertia ixx="0.00017957425901848" ixy="6.28960386226657E-21" ixz="2.14010788664762E-21"
+                iyy="0.00017957425901848" iyz="1.27709655724716E-22" izz="0.000332594534732139" />
         </inertial>
         <visual>
@@ -218,5 +232,7 @@
             <origin xyz="3.51083051564616E-05 -2.7181014665284E-05 0.0709276770204769" rpy="0 0 0" />
             <mass value="0.240893303086836" />
-            <inertia ixx="0.000105035118852508" ixy="1.32328029886296E-08" ixz="3.84294589110161E-11" iyy="0.00010502957299471" iyz="-1.41155611875745E-11" izz="0.00017298179736849" />
+            <inertia ixx="0.000105035118852508" ixy="1.32328029886296E-08"
+                ixz="3.84294589110161E-11"
+                iyy="0.00010502957299471" iyz="-1.41155611875745E-11" izz="0.00017298179736849" />
         </inertial>
         <visual>
@@ -244,5 +260,7 @@
             <origin xyz="-1.5143569731535E-10 7.07767178198537E-16 -0.0246054820762604" rpy="0 0 0" />
             <mass value="1.35828296445862" />
-            <inertia ixx="0.00232456013775523" ixy="-1.61343020248111E-09" ixz="-4.5670735364335E-13" iyy="0.00232456564213727" iyz="-1.36036258272812E-18" izz="0.00308347787030649" />
+            <inertia ixx="0.00232456013775523" ixy="-1.61343020248111E-09"
+                ixz="-4.5670735364335E-13"
+                iyy="0.00232456564213727" iyz="-1.36036258272812E-18" izz="0.00308347787030649" />
         </inertial>
         <visual>
@@ -270,5 +288,7 @@
             <origin xyz="5.55111512312578E-17 5.55111512312578E-17 -0.0720000000000002" rpy="0 0 0" />
             <mass value="0.271192811687251" />
-            <inertia ixx="0.000179574259018481" ixy="-1.73824343982442E-20" ixz="-2.53159654382751E-21" iyy="0.000179574259018481" iyz="-3.13741449878515E-21" izz="0.000332594534732139" />
+            <inertia ixx="0.000179574259018481" ixy="-1.73824343982442E-20"
+                ixz="-2.53159654382751E-21"
+                iyy="0.000179574259018481" iyz="-3.13741449878515E-21" izz="0.000332594534732139" />
         </inertial>
         <visual>
@@ -296,5 +316,6 @@
             <origin xyz="7.58128369110489E-17 7.63278329429795E-17 -0.0720000000000003" rpy="0 0 0" />
             <mass value="0.27119281168725" />
-            <inertia ixx="0.00017957425901848" ixy="9.82929052458426E-22" ixz="1.10990388135291E-21" iyy="0.00017957425901848" iyz="-4.81322327079121E-21" izz="0.000332594534732139" />
+            <inertia ixx="0.00017957425901848" ixy="9.82929052458426E-22" ixz="1.10990388135291E-21"
+                iyy="0.00017957425901848" iyz="-4.81322327079121E-21" izz="0.000332594534732139" />
         </inertial>
         <visual>
@@ -322,5 +343,7 @@
             <origin xyz="1.37732703020532E-08 -5.29206664124648E-05 -0.0701501700151683" rpy="0 0 0" />
             <mass value="0.245836054976119" />
-            <inertia ixx="0.000105264944409738" ixy="7.98231761628902E-12" ixz="6.80400273605472E-11" iyy="0.000105238344260685" iyz="-2.72106317781962E-11" izz="0.000173281039335396" />
+            <inertia ixx="0.000105264944409738" ixy="7.98231761628902E-12"
+                ixz="6.80400273605472E-11"
+                iyy="0.000105238344260685" iyz="-2.72106317781962E-11" izz="0.000173281039335396" />
         </inertial>
         <visual>
@@ -348,5 +371,7 @@
             <origin xyz="5.55111512312578E-17 1.51436273243544E-10 0.0245928853369881" rpy="0 0 0" />
             <mass value="1.35828296445862" />
-            <inertia ixx="0.00232456564213727" ixy="-1.6134302023684E-09" ixz="-3.67391703208082E-19" iyy="0.00232456013775523" iyz="-4.56707494796216E-13" izz="0.00308347787030649" />
+            <inertia ixx="0.00232456564213727" ixy="-1.6134302023684E-09"
+                ixz="-3.67391703208082E-19"
+                iyy="0.00232456013775523" iyz="-4.56707494796216E-13" izz="0.00308347787030649" />
         </inertial>
         <visual>
@@ -374,5 +399,7 @@
             <origin xyz="-1.11022302462516E-16 -5.55111512312578E-17 0.0720000000000002" rpy="0 0 0" />
             <mass value="0.271192811687251" />
-            <inertia ixx="0.000179574259018481" ixy="-7.93399024302093E-21" ixz="-2.13342044570487E-21" iyy="0.000179574259018481" iyz="-3.23624373974149E-21" izz="0.000332594534732139" />
+            <inertia ixx="0.000179574259018481" ixy="-7.93399024302093E-21"
+                ixz="-2.13342044570487E-21"
+                iyy="0.000179574259018481" iyz="-3.23624373974149E-21" izz="0.000332594534732139" />
         </inertial>
         <visual>
@@ -400,5 +427,6 @@
             <origin xyz="-7.64498056873841E-17 -4.85722573273506E-17 0.0720000000000004" rpy="0 0 0" />
             <mass value="0.27119281168725" />
-            <inertia ixx="0.00017957425901848" ixy="6.3005828905746E-22" ixz="1.1753358195074E-22" iyy="0.00017957425901848" iyz="-3.27347099653111E-21" izz="0.000332594534732139" />
+            <inertia ixx="0.00017957425901848" ixy="6.3005828905746E-22" ixz="1.1753358195074E-22"
+                iyy="0.00017957425901848" iyz="-3.27347099653111E-21" izz="0.000332594534732139" />
         </inertial>
         <visual>
@@ -426,5 +454,7 @@
             <origin xyz="1.37732700244975E-08 -5.29206664124926E-05 0.0701152686893121" rpy="0 0 0" />
             <mass value="0.245836054976119" />
-            <inertia ixx="0.000105264944409738" ixy="7.98231761858719E-12" ixz="6.80400273764357E-11" iyy="0.000105238344260685" iyz="-2.72106317797361E-11" izz="0.000173281039335396" />
+            <inertia ixx="0.000105264944409738" ixy="7.98231761858719E-12"
+                ixz="6.80400273764357E-11"
+                iyy="0.000105238344260685" iyz="-2.72106317797361E-11" izz="0.000173281039335396" />
         </inertial>
         <visual>
@@ -1508,5 +1538,6 @@
     <!-- Bunker new plugins -->
     <gazebo>
-        <plugin filename="gz-sim-joint-state-publisher-system" name="gz::sim::systems::JointStatePublisher">
+        <plugin filename="libignition-gazebo-joint-state-publisher-system.so"
+            name="ignition::gazebo::systems::JointStatePublisher">
             <topic>joint_states</topic>
             <update_rate>50</update_rate>
@@ -1534,5 +1565,6 @@
             <joint_name>right_track_rear_wheel1_j</joint_name>
         </plugin>
-        <plugin filename="gz-sim-diff-drive-system" name="gz::sim::systems::DiffDrive">
+        <plugin filename="libignition-gazebo-diff-drive-system.so"
+            name="ignition::gazebo::systems::DiffDrive">
             <left_joint>left_track_wheel0_j</left_joint>
             <right_joint>right_track_wheel0_j</right_joint>

File: scout/scout_description/urdf/scout_mini.xacro (robot description, xacro)
@@ -1,5 +1,4 @@
 <?xml version="1.0"?>
-<robot name="scout_mini"
-    xmlns:xacro="http://ros.org/wiki/xacro">
+<robot name="scout_mini" xmlns:xacro="http://ros.org/wiki/xacro">
     <!-- Vehicle Geometries -->
     <!-- Base link -->
@@ -8,5 +7,6 @@
             <origin xyz="0 0 0" rpy="1.57 0 -1.57" />
             <geometry>
-                <mesh filename="package://scout_description/meshes/scout_mini_base_link.dae" />
+                <mesh
+                    filename="package://scout_description/meshes/scout_mini_base_link.dae" />
             </geometry>
         </visual>
@@ -14,16 +14,20 @@
             <origin xyz="0 0 0" rpy="1.57 0 -1.57" />
             <geometry>
-                <mesh filename="package://scout_description/meshes/scout_mini_base_link.dae" />
+                <mesh
+                    filename="package://scout_description/meshes/scout_mini_base_link.dae" />
             </geometry>
         </collision>
     </link>
-    <link name="inertial_link">
+    <link
+        name="inertial_link">
         <inertial>
             <mass value="132.3898489950015" />
             <origin xyz=" 0 0 0" />
-            <inertia ixx="0.185196122711036" ixy="4.30144213829512E-08" ixz="5.81037523686401E-08" iyy="0.364893736238929" iyz="-0.000386720198091934" izz="0.223868521722778" />
+            <inertia ixx="0.185196122711036" ixy="4.30144213829512E-08" ixz="5.81037523686401E-08"
+                iyy="0.364893736238929" iyz="-0.000386720198091934" izz="0.223868521722778" />
         </inertial>
     </link>
-    <joint name="inertial_joint" type="fixed">
+    <joint
+        name="inertial_joint" type="fixed">
         <origin xyz="0 0 0" rpy="0 0 0" />
         <parent link="base_link" />
@@ -31,5 +35,6 @@
     </joint>
     <!-- Scout wheel -->
-    <link name="front_right_wheel_link">
+    <link
+        name="front_right_wheel_link">
         <inertial>
             <mass value="3" />
@@ -50,5 +55,6 @@
         </collision>
     </link>
-    <joint name="front_right_wheel" type="continuous">
+    <joint
+        name="front_right_wheel" type="continuous">
         <origin rpy="1.57 0 0" xyz="0.2319755 -0.2082515 -0.099998" />
         <parent link="base_link" />
@@ -75,5 +81,6 @@
         </collision>
     </link>
-    <joint name="front_left_wheel" type="continuous">
+    <joint
+        name="front_left_wheel" type="continuous">
         <origin rpy="-1.57 0 0" xyz="0.2319755 0.2082515 -0.100998" />
         <parent link="base_link" />
@@ -100,5 +107,6 @@
         </collision>
     </link>
-    <joint name="rear_right_wheel" type="continuous">
+    <joint
+        name="rear_right_wheel" type="continuous">
         <origin rpy="1.57 0 0" xyz="-0.2319755 -0.2082515 -0.099998" />
         <parent link="base_link" />
@@ -125,5 +133,6 @@
         </collision>
     </link>
-    <joint name="rear_left_wheel" type="continuous">
+    <joint
+        name="rear_left_wheel" type="continuous">
         <origin rpy="-1.57 0 0" xyz="-0.2319755 0.2082515 -0.100998" />
         <parent link="base_link" />
@@ -133,5 +142,6 @@
     <!-- Scout gazebo plugin -->
     <gazebo>
-        <plugin filename="gz-sim-joint-state-publisher-system" name="gz::sim::systems::JointStatePublisher">
+        <plugin filename="libignition-gazebo-joint-state-publisher-system.so"
+            name="ignition::gazebo::systems::JointStatePublisher">
             <topic>joint_states</topic>
             <update_rate>50</update_rate>
@@ -141,5 +151,7 @@
             <joint_name>rear_left_wheel</joint_name>
         </plugin>
-        <plugin filename="gz-sim-diff-drive-system" name="gz::sim::systems::DiffDrive">
+        <plugin
+            filename="libignition-gazebo-diff-drive-system.so"
+            name="ignition::gazebo::systems::DiffDrive">
             <left_joint>front_left_wheel</left_joint>
             <right_joint>front_right_wheel</right_joint>
